File: Column Staggered Variant Files/PCB/CurvedChoc/CurvedChoc.sch (KiCad schematic (older format))
At the start: 48 parts, among them SW1 2-Pos, SW10 Switch, SW11 Switch, SW12 Switch, SW13 Switch, SW14 Switch, SW15 Switch, SW16 Switch, SW17 Switch, SW18 REsw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

Commit message: Updated to include Rev2 QMK and Gerbers
Parts:
- added M1: MouseBite, KeyboardFootprints:Mousebite, symbol KeyboardLibrary:MouseBite
- H1, H2, H3, H4, H5: footprint KeyboardFootprints:MountingHole_2.9mm -> KeyboardFootprints:Hole_2mm
- SW18: symbol KeyboardLibrary:REsw -> CurvedChoc-rescue:REsw-KeyboardLibrary
Changed lines of the file:
@@
 E2
 $Comp
-L KeyboardLibrary:REsw SW18
+L CurvedChoc-rescue:REsw-KeyboardLibrary SW18
 U 1 1 5EF24DCA
 P 6150 3500
@@
 F 0 "H1" H 10250 900 50  0000 C CNN
 F 1 "Hole" H 10250 1100 50  0000 C CNN
-F 2 "KeyboardFootprints:MountingHole_2.9mm" H 10250 950 50  0001 C CNN
+F 2 "KeyboardFootprints:Hole_2mm" H 10250 950 50  0001 C CNN
 F 3 "" H 10250 950 50  0001 C CNN
 	1    10250 1000
@@
 F 0 "H2" H 10550 900 50  0000 C CNN
 F 1 "Hole" H 10550 1100 50  0000 C CNN
-F 2 "KeyboardFootprints:MountingHole_2.9mm" H 10550 950 50  0001 C CNN
+F 2 "KeyboardFootprints:Hole_2mm" H 10550 950 50  0001 C CNN
 F 3 "" H 10550 950 50  0001 C CNN
 	1    10550 1000
@@
 F 0 "H3" H 10400 1150 50  0000 C CNN
 F 1 "Hole" H 10400 1350 50  0000 C CNN
-F 2 "KeyboardFootprints:MountingHole_2.9mm" H 10400 1200 50  0001 C CNN
+F 2 "KeyboardFootprints:Hole_2mm" H 10400 1200 50  0001 C CNN
 F 3 "" H 10400 1200 50  0001 C CNN
 	1    10400 1250
@@
 F 0 "H4" H 10250 1400 50  0000 C CNN
 F 1 "Hole" H 10250 1600 50  0000 C CNN
-F 2 "KeyboardFootprints:MountingHole_2.9mm" H 10250 1450 50  0001 C CNN
+F 2 "KeyboardFootprints:Hole_2mm" H 10250 1450 50  0001 C CNN
 F 3 "" H 10250 1450 50  0001 C CNN
 	1    10250 1500
@@
 F 0 "H5" H 10550 1400 50  0000 C CNN
 F 1 "Hole" H 10550 1600 50  0000 C CNN
-F 2 "KeyboardFootprints:MountingHole_2.9mm" H 10550 1450 50  0001 C CNN
+F 2 "KeyboardFootprints:Hole_2mm" H 10550 1450 50  0001 C CNN
 F 3 "" H 10550 1450 50  0001 C CNN
 	1    10550 1500
@@
 	6850 3400 6850 2800
 Connection ~ 6850 2800
+$Comp
+L KeyboardLibrary:MouseBite M1
+U 1 1 5EF3C917
+P 10100 2000
+F 0 "M1" H 10100 2100 50  0000 C CNN
+F 1 "MouseBite" H 10100 1900 50  0000 C CNN
+F 2 "KeyboardFootprints:Mousebite" H 10100 2000 50  0001 C CNN
+F 3 "" H 10100 2000 50  0001 C CNN
+	1    10100 2000
+	1    0    0    -1
+$EndComp
 $EndSCHEMATC
